Commit message: Haokun

File: robots/mini_quadrotor/urdf/robot.urdf.xacro (robot description, xacro)
@@ -36,4 +36,50 @@
       </xacro:if>
     </link>
+  </xacro:macro>
+  <xacro:macro name="extra_camera" params="name parent *origin *inertial visible:=0 model_url:=1 scale:=1">
+    <joint name="${parent}2${name}" type="fixed">
+      <parent link="${parent}"/>
+      <child link="${name}"/>
+      <xacro:insert_block name="origin" />
+    </joint>
+    <link name="${name}">
+      <xacro:insert_block name="inertial" />
+      <xacro:if value="${visible == 1}">
+        <visual>
+          <origin rpy="0 0 0" xyz="0 0 0"/>
+          <geometry>
+            <mesh filename="${model_url}" scale= "${scale} ${scale} ${scale}"/>
+          </geometry>
+        </visual>
+      </xacro:if>
+      <!-- Camera Sensor Definition for Gazebo -->
+    </link>
+    <gazebo reference="${name}">
+      <sensor type="camera" name="camera_sensor">
+        <update_rate>30.0</update_rate>
+        <camera>
+          <horizontal_fov>1.047</horizontal_fov>
+          <image>
+            <width>1280</width>
+            <height>960</height>
+            <format>R8G8B8</format>
+          </image>
+          <clip>
+            <near>0.1</near>
+            <far>100</far>
+          </clip>
+        </camera>
+        <always_on>true</always_on>
+        <visualize>true</visualize>
+        <plugin name="camera_controller" filename="libgazebo_ros_camera.so">
+          <alwaysOn>true</alwaysOn>
+          <updateRate>5</updateRate>
+          <cameraName>high_altitude_camera</cameraName>
+          <imageTopicName>/camera/image_raw</imageTopicName>
+          <cameraInfoTopicName>/camera/camera_info</cameraInfoTopicName>
+          <frameName>${name}_link</frameName>
+        </plugin>
+      </sensor>
+    </gazebo>
   </xacro:macro>
   <xacro:macro name="propeller_module" params="id x y z direction">
@@ -149,4 +195,15 @@
     </inertial>
   </xacro:extra_module>
+  <!-- camera module -->
+  <xacro:extra_camera name="camera" parent="main_body" visible="1" model_url = "package://mini_quadrotor/urdf/mesh/realsense.dae">
+    <origin xyz="0.0 0 -0.05" rpy="0 ${pi/2} 0"/>
+    <inertial>
+      <mass value="0.1"/>
+      <origin xyz="0 0 0" rpy="0 0 0"/>
+      <inertia
+          ixx="0.0001" ixy="0.0" ixz="0.0"
+          iyy="0.0001" iyz="0.0" izz="0.0001"/>
+    </inertial>
+  </xacro:extra_camera>
   <!-- propellers -->
   <xacro:propeller_module id = "1" x = "${-rotor_x}" y = "${-rotor_y}" z = "${rotor_z}" direction = "-1" />
