Commit message: Add shell_link and shell_joint to go1.urdf

File: robots/go1_description/urdf/go1.urdf (robot description, URDF)
Before this commit: robot go1, 46 links, 45 joints
Links:
- added link shell_link; visual box size=0.6 0.6 0.2
Joints:
- added joint shell_joint: type fixed, parent trunk, child shell_link, origin xyz=0 0 0.1 rpy=0 0 0

File: robots/go1_description/xacro/materials.xacro (robot description, xacro)
@@ -24,4 +24,5 @@
     <material name="red">
         <color rgba="0.8 0.0 0.0 1.0"/>
+        <ambient rgba="0.4 0.0 0.0 1.0"/>
     </material>
     <material name="white">

File: robots/go1_description/xacro/robot.xacro (robot description, xacro)
@@ -3,5 +3,5 @@
     <xacro:arg name="DEBUG" default="false"/>
     <xacro:include filename="$(find go1_description)/xacro/const.xacro"/>
-    <xacro:include filename="$(find go1_description)/xacro/materials.xacro"/>
+    <!-- <xacro:include filename="$(find go1_description)/xacro/materials.xacro"/> -->
     <xacro:include filename="$(find go1_description)/xacro/leg.xacro"/>
     <!-- <xacro:include filename="$(find go1_description)/xacro/stairs.xacro"/> -->
@@ -10,4 +10,8 @@
     <xacro:include filename="$(find go1_description)/xacro/ultraSound.xacro"/>
     <!-- <xacro:include filename="$(find go1_gazebo)/launch/stairs.urdf.xacro"/> -->
+    <material name="red">
+        <color rgba="0.8 0.0 0.0 1.0"/>
+        <ambient rgba="0.4 0.0 0.0 1.0"/>
+    </material>
     <!-- <xacro:stairs stairs="15" xpos="0" ypos="0" zpos="0" /> -->
     <!-- Rotor related joint and link is only for demonstrate location. -->
@@ -58,4 +62,46 @@
         </inertial>
     </link>
+    <joint name="front_joint" type="fixed">
+        <parent link="trunk"/>
+        <child link="front_link"/>
+        <origin xyz="0 0 0.1" rpy="0 0 0"/>
+    </joint>
+    <link name="front_link">
+        <visual>
+            <origin xyz="-0.1 0 -0.03" rpy="0 0 0"/>
+            <geometry>
+                <box size="0.1 0.2 0.02"/>
+            </geometry>
+            <material name="custom_red">
+                <color rgba="0.851 0.0 0.0 1.0"/>
+            </material>
+        </visual>
+    </link>
+    <gazebo reference="front_link">
+        <material>
+            Gazebo/Red
+        </material>
+    </gazebo>
+    <joint name="rear_joint" type="fixed">
+        <parent link="trunk"/>
+        <child link="rear_link"/>
+        <origin xyz="0 0 0.1" rpy="0 0 0"/>
+    </joint>
+    <link name="rear_link">
+        <visual>
+            <origin xyz="0.18 0 -0.03" rpy="0 0 0"/>
+            <geometry>
+                <box size="0.2 0.05 0.02"/>
+            </geometry>
+            <material name="custom_red">
+                <color rgba="0.851 0.0 0.0 1.0"/>
+            </material>
+        </visual>
+    </link>
+    <gazebo reference="rear_link">
+        <material>
+            Gazebo/Black
+        </material>
+    </gazebo>
     <joint name="imu_joint" type="fixed">
         <parent link="trunk"/>
